File: revision0/revision0.kicad_sch (KiCad schematic)
At the start: 36 parts, among them J1 USB1, J10 Conn_01x03, J2 Conn_01x07, J3 Conn_02x03_Counter_Clockwise, J4 Conn_01x05, J5 Conn_02x03_Counter_Clockwise, J6 Conn_02x03_Counter_Clockwise, J7 Conn_02x03_Counter_Clockwise, J8 Conn_01x04, J9 Conn_01x03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

Commit message: minor fix
Parts:
- removed D8: CLX6F-FKC, LED_SMD:LED_RGB_PLCC-6, symbol LED:CLX6F-FKC
- removed J10: Conn_01x03, Connector_PinHeader_2.54mm:PinHeader_1x03_P2.54mm_Vertical, symbol Connector_Generic:Conn_01x03
- removed R9: 1k, Resistor_SMD:R_0805_2012Metric_Pad1.20x1.40mm_HandSolder, symbol Device:R

Commit message: update project w/ missing footprint
Parts:
- J1: footprint Library:USB_A_Molex_67643_Horizontal -> usb:USB_A_Molex_67643_Horizontal
Changed lines of the file:
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@@
 			)
 		)
-		(property "Footprint" "Library:USB_A_Molex_67643_Horizontal"
+		(property "Footprint" "usb:USB_A_Molex_67643_Horizontal"
 			(at 209.55 88.9 0)
 			(effects
